Commit message: more progress

File: urdf/LeKiwi.urdf (robot description, URDF)
Before this commit: robot LeKiwi, 45 links, 44 joints
Links:
- removed link Moving_Jaw_08d-v1
- removed link Wrist_Roll_08c-v1
- added link Fixed_Jaw, mass 0.44698022927880193; collision mesh filename=meshes/Wrist_Roll_08c-v1.stl scale=0.001 0.001 0.001; visual mesh filename=meshes/Wrist_Roll_08c-v1.stl scale=0.001 0.001 0.001
- added link Fixed_Jaw_tip
- added link Moving_Jaw, mass 0.1586808414280307; collision mesh filename=meshes/Moving_Jaw_08d-v1.stl scale=0.001 0.001 0.001; visual mesh filename=meshes/Moving_Jaw_08d-v1.stl scale=0.001 0.001 0.001
- added link Moving_Jaw_tip
- added link root, mass 0
- added link root_arm_1_link_1, mass 0
- added link root_arm_1_link_2, mass 0
Joints:
- added joint Fixed_Jaw_tip_joint: type fixed, parent Fixed_Jaw, child Fixed_Jaw_tip, origin xyz=0.01 -0.097 0 rpy=0 0 0
- added joint Moving_Jaw_tip_joint: type fixed, parent Moving_Jaw, child Moving_Jaw_tip, origin xyz=-0.01 -0.073 0 rpy=0 0 0
- added joint root_x_axis_joint: type prismatic, parent root, child root_arm_1_link_1, axis 1 0 0, limit lower=-20 upper=20 effort=100 velocity=0.50
- added joint root_y_axis_joint: type prismatic, parent root_arm_1_link_1, child root_arm_1_link_2, axis 0 1 0, limit lower=-20 upper=20 effort=100 velocity=0.50
- added joint root_z_rotation_joint: type continuous, parent root_arm_1_link_2, child base_link, axis 0 0 1
- joint Wrist_Roll_08c-v1_Rigid-56: parent Wrist_Roll_08c-v1 -> Fixed_Jaw
- joint Wrist_Roll_08c-v1_Rigid-58: parent Wrist_Roll_08c-v1 -> Fixed_Jaw
- joint elbow_flex: limit (none) -> lower=-1.5708 upper=1.5708 effort=0 velocity=0
- joint gripper: child Moving_Jaw_08d-v1 -> Moving_Jaw; limit (none) -> lower=-1.1 upper=1.1 effort=0 velocity=0
- joint shoulder_lift: limit (none) -> lower=-1.5708 upper=1.5708 effort=0 velocity=0
- joint shoulder_pan: limit (none) -> lower=-2.0 upper=2.0 effort=0 velocity=0
- joint wrist_flex: limit (none) -> lower=-1.8 upper=1.8 effort=0 velocity=0
- joint wrist_roll: child Wrist_Roll_08c-v1 -> Fixed_Jaw; limit (none) -> lower=-3.14159 upper=3.14159 effort=0 velocity=0

File: urdf/custom_lekiwi.urdf (robot description, URDF)
Before this commit: robot SO_5DOF_ARM100_8j_URDF.SLDASM, 9 links, 8 joints
Joints:
- added joint arm_base_joint: type fixed, parent base_plate_layer2-v3, child Base, origin xyz=0.04 0.08 0.007 rpy=0 0 0

Commit message: urdf looking good

File: urdf/LeKiwi.urdf (robot description, URDF)
Before this commit: robot LeKiwi, 50 links, 49 joints
Links:
- removed link base_plate_layer1-v5
- added link base_link, mass 1.9468624348344596; collision mesh filename=meshes/base_plate_layer1-v5.stl scale=0.001 0.001 0.001; visual mesh filename=meshes/base_plate_layer1-v5.stl scale=0.001 0.001 0.001
Joints:
- joint ST3215_Servo_Motor-v1-1_Revolute-62: type continuous -> fixed
- joint ST3215_Servo_Motor-v1-2_Revolute-60: type continuous -> fixed
- joint ST3215_Servo_Motor-v1_Revolute-64: type continuous -> fixed
- joint base_plate_layer1-v5_Rigid-15: parent base_plate_layer1-v5 -> base_link
- joint base_plate_layer1-v5_Rigid-18: parent base_plate_layer1-v5 -> base_link
- joint base_plate_layer1-v5_Rigid-20: parent base_plate_layer1-v5 -> base_link
- joint base_plate_layer1-v5_Rigid-28: parent base_plate_layer1-v5 -> base_link
- joint base_plate_layer1-v5_Rigid-30: parent base_plate_layer1-v5 -> base_link
- joint base_plate_layer1-v5_Rigid-31: parent base_plate_layer1-v5 -> base_link
- joint base_plate_layer1-v5_Rigid-32: parent base_plate_layer1-v5 -> base_link
- joint base_plate_layer1-v5_Rigid-69: parent base_plate_layer1-v5 -> base_link
- joint base_plate_layer1-v5_Rigid-70: parent base_plate_layer1-v5 -> base_link
- joint base_plate_layer1-v5_baseplate2bottom_mount: parent base_plate_layer1-v5 -> base_link
- joint base_plate_layer1-v5_baseplate2left_mount: parent base_plate_layer1-v5 -> base_link
- joint base_plate_layer1-v5_baseplate2right_mount: parent base_plate_layer1-v5 -> base_link
- joint root_z_rotation_joint: origin (none) -> xyz=0 0 0.036 rpy=0 0 0

Commit message: gain tuning

File: urdf/LeKiwi.urdf (robot description, URDF)
Before this commit: robot LeKiwi, 50 links, 49 joints
Joints:
- joint base_plate_layer1-v5_Rigid-28: origin xyz=0.02 0.1 0.0 rpy=0.0 -0.0 0.0 -> xyz=0.02 0.1 0.0 rpy=0.0 -0.0 1.57
- joint root_z_rotation_joint: origin xyz=0 0 0.036 rpy=0 0 0 -> xyz=0 0 0.015 rpy=0 0 0

Commit message: working lekiwi teleopgit add .

File: urdf/LeKiwi.urdf (robot description, URDF)
Before this commit: robot LeKiwi, 50 links, 49 joints
Joints:
- joint root_x_axis_joint: axis 1 0 0 -> 0 1 0; child root_arm_1_link_1 -> root_arm_1_link_2; parent root -> root_arm_1_link_1
- joint root_y_axis_joint: axis 0 1 0 -> -1 0 0; child root_arm_1_link_2 -> root_arm_1_link_1; parent root_arm_1_link_1 -> root
- joint shoulder_pan: limit lower=-2.0 upper=2.0 effort=0 velocity=0 -> (none); type continuous -> fixed
